File: KiCad_src_V1_2/KiCad_src_V1_2.kicad_pcb (KiCad board)
At the start: 4 copper layers, 74.1 x 130 mm, 132 parts, among them J1 USB_C_Receptacle_USB2.0_14P, J4 AFC07-S24ECA-00, J5 Micro_SD_Card_Det1, Q1 2N7002, Q2 SI1308EDL, Q3 SI2301, SW1 TS-1187A-B-A-B, SW2 K2-1112SW-A4SW-04, SW3 K2-1112SW-A4SW-04, SW4 XDTD-6650, SW5 XDTD-6650, SW6 TS-1187A-B-A-B, SW7 SW_SPDT, U1 RP2040, U2 74HC139, U3 W25Q128JVSIQ, U4 CC1101RGPR, U5 TP4056, U6 TPS63000, U7 LM321, X1 ABM8-272-T3, X2 26MHz

Commit message: Add production preview documentation and associated files for JLCPCB order
Routing:
- net GND: vias 196 -> 1225
