File: KiCad_src_V1_2/KiCad_src_V1_2.kicad_sch (KiCad schematic)
At the start: 132 parts, among them J1 USB_C_Receptacle_USB2.0_14P, J4 AFC07-S24ECA-00, J5 Micro_SD_Card_Det1, Q1 2N7002, Q2 SI1308EDL, Q3 SI2301, SW1 TS-1187A-B-A-B, SW2 K2-1112SW-A4SW-04, SW3 K2-1112SW-A4SW-04, SW4 XDTD-6650, SW5 XDTD-6650, SW6 TS-1187A-B-A-B, SW7 SW_SPDT, U1 RP2040, U2 74HC139, U3 W25Q128JVSIQ, U4 CC1101RGPR, U5 TP4056, U6 TPS63000, U7 LM321, X1 ABM8-272-T3, X2 26MHz

Commit message: Library for inverted F antenna added (need more room on PCB). Capacitor components changed to C0G
Parts:
- C21, C26: LCSC Part # C1530 -> C71693; Manufacturer FH -> MURATA; Manufacturer Part 0402B221K500NT -> GRM1555C1H221JA01D; Supplier Part C1530 -> C71693
Changed lines of the file:
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@@
 			)
 		)
-		(property "Manufacturer" "FH"
+		(property "Manufacturer" "MURATA"
 			(at 355.6 171.45 0)
 			(hide yes)
@@
 			)
 		)
-		(property "Manufacturer Part" "0402B221K500NT"
+		(property "Manufacturer Part" "GRM1555C1H221JA01D"
 			(at 355.6 171.45 0)
 			(hide yes)
@@
 			)
 		)
-		(property "Supplier Part" "C1530"
+		(property "Supplier Part" "C71693"
 			(at 355.6 171.45 0)
 			(hide yes)
@@
 			)
 		)
-		(property "LCSC Part #" "C1530"
+		(property "LCSC Part #" "C71693"
 			(at 355.6 171.45 0)
 			(hide yes)
@@
 			)
 		)
-		(property "Manufacturer" "FH"
+		(property "Manufacturer" "MURATA"
 			(at 316.23 156.21 0)
 			(hide yes)
@@
 			)
 		)
-		(property "Manufacturer Part" "0402B221K500NT"
+		(property "Manufacturer Part" "GRM1555C1H221JA01D"
 			(at 316.23 156.21 0)
 			(hide yes)
@@
 			)
 		)
-		(property "Supplier Part" "C1530"
+		(property "Supplier Part" "C71693"
 			(at 316.23 156.21 0)
 			(hide yes)
@@
 			)
 		)
-		(property "LCSC Part #" "C1530"
+		(property "LCSC Part #" "C71693"
 			(at 316.23 156.21 0)
 			(hide yes)
